File: de1-sdr.kicad_sch (KiCad schematic)
At the start: 176 parts, among them J1 RF IN, J2 DE1-HEADER, J3 UFL, Q1 BSS138, Q2 AO3401A, T1 TC4-1TX+, U1 AD9609-40, U10 TPS7A2018DBV, U11 TPS7A2030DBV, U12 TPS7A2030DBV, U13 TPS7A2030DBV, U2 QPL9547, U3 MAX2862, U4 LMX2594, U5 BDA4620, U6 TPS7A2018DBV, U7 PAT1220-C-2DB, U8 BG18C, U9 BG18C, Y1 ECS-3518-800-B-TR

Commit message: fix erc
Connections:
- no-connect marks 14 -> 19
Other:
- moved on the sheet: C72, C73, C74, C75, C82, C83, C84, C85, FB10, FB14, FB15, FB9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

Commit message: fixed typos
Parts:
- added FL3: B39162B8813P810, Filter:Filter_1109-5_1.1x0.9mm, symbol Filter:B39162B8813P810
- added R45, R46: 1k, Resistor_SMD:R_0402_1005Metric, symbol Device:R_Small
- added R47, R48: 100k, Resistor_SMD:R_0402_1005Metric, symbol Device:R_Small
- U1: value AD9609-40 -> AD9609-80
- U11, U12, U13: value TPS7A2030DBV -> TPS7A2033DBV
- U3: value MAX2862 -> MAX2682
Connections:
- net +3V3_ANT: now also R48.1
- net ANT_PWR_EN: now also R48.2
- net GND: now also FL3.2, FL3.3, FL3.5, R46.2, R47.1
- net LNA_EN: now also R47.2
- net XO_EN: now also R45.2; no longer Y1.1 (Tri-State)
- net at U5.2 (RF1): now also FL3.4; no longer C12.2
- new net: R45.1, R46.1, Y1.1 (Tri-State)
- new net: C12.2, FL3.1
Other:
- moved on the sheet: C10, C11, C12, C13, C14, C15, C18, C19, FL1, J1, L6, L7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

Commit message: fix more typo
Parts:
- U4: value LMX2594 -> LMX2572
Changed lines of the file:
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@@
 	(text_box "Gain block and balun"
 		(exclude_from_sim no)
-		(at 393.7 129.4017 0)
-		(size 25.4 3.9483)
+		(at 393.7 129.54 0)
+		(size 26.67 5.2183)
 		(margins 0.9525 0.9525 0.9525 0.9525)
 		(stroke
@@
 			)
 		)
-		(property "Value" "LMX2594"
+		(property "Value" "LMX2572"
 			(at 164.7033 334.01 0)
 			(show_name no)
@@
 			)
 		)
-		(property "Datasheet" "https://www.ti.com/lit/ds/symlink/lmx2594.pdf"
+		(property "Datasheet" ""
 			(at 154.94 302.26 0)
 			(hide yes)
@@
 			)
 		)
-		(property "Description" "LMX2594 15-GHz Wideband PLLATINUM™ RF Synthesizer With Phase Synchronization and JESD204B Support"
+		(property "Description" ""
 			(at 154.94 302.26 0)
 			(hide yes)

Commit message: fix more typo
Parts:
- U4: footprint Package_DFN_QFN:VQFN-40-1EP_6x6mm_P0.5mm_EP3.5x3.5mm_ThermalVias -> Package_DFN_QFN:HVQFN-40-1EP_6x6mm_P0.5mm_EP4.1x4.1mm
Changed lines of the file:
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@@
 		(exclude_from_sim no)
 		(at 393.7 129.54 0)
-		(size 26.67 5.2183)
+		(size 26.67 3.9483)
 		(margins 0.9525 0.9525 0.9525 0.9525)
 		(stroke
@@
 	(text_box "-82.5 dBm"
 		(exclude_from_sim no)
-		(at 240.03 86.2217 0)
+		(at 240.03 84.9517 0)
 		(size 13.97 3.9483)
 		(margins 0.9525 0.9525 0.9525 0.9525)
@@
 			)
 		)
-		(property "Footprint" "Package_DFN_QFN:VQFN-40-1EP_6x6mm_P0.5mm_EP3.5x3.5mm_ThermalVias"
+		(property "Footprint" "Package_DFN_QFN:HVQFN-40-1EP_6x6mm_P0.5mm_EP4.1x4.1mm"
 			(at 154.94 302.26 0)
 			(hide yes)
@@
 			)
 		)
-		(property "Datasheet" ""
+		(property "Datasheet" "https://www.ti.com/lit/ds/symlink/lmx2572.pdf"
 			(at 154.94 302.26 0)
 			(hide yes)
@@
 			)
 		)
-		(property "Description" ""
+		(property "Description" "LMX2572 6.4-GHz Low power wideband RF synthesizer with phase synchronization and JESD204B support"
 			(at 154.94 302.26 0)
 			(hide yes)

Commit message: added lc filter parts
Parts:
- removed C4: C_Small, symbol Device:C_Small
- added L10: 56n, Inductor_SMD:L_1008_2520Metric, symbol Device:L_Small
- added L13: 160n, Inductor_SMD:L_0805_2012Metric, symbol Device:L_Small
- C1: value C_Small -> 130p; footprint (none) -> Capacitor_SMD:C_0402_1005Metric
- C2: value C_Small -> 8.5p; footprint (none) -> Capacitor_SMD:C_0402_1005Metric
- C3: value C_Small -> 47p; footprint (none) -> Capacitor_SMD:C_0402_1005Metric
- C5: value C_Small -> 150p; footprint (none) -> Capacitor_SMD:C_0402_1005Metric
- C6: value C_Small -> 7.1p; footprint (none) -> Capacitor_SMD:C_0402_1005Metric
- C66: value 390p -> 1.5n; now fitted
- C67: value 15n -> 220n
- C68: value 300p -> (none)
- C69: value 2.2n -> (none); now not fitted
- C7: value C_Small -> 16p; footprint (none) -> Capacitor_SMD:C_0402_1005Metric
- C8: value C_Small -> 82p; footprint (none) -> Capacitor_SMD:C_0402_1005Metric
- C9: value C_Small -> 160p; footprint (none) -> Capacitor_SMD:C_0402_1005Metric
- L1: value L_Small -> 20n; footprint (none) -> Inductor_SMD:L_0805_2012Metric
- L2: value L_Small -> 300n; footprint (none) -> Inductor_SMD:L_1008_2520Metric
- L3: value L_Small -> 11n; footprint (none) -> Inductor_SMD:L_0805_2012Metric
- L4: value L_Small -> 360n; footprint (none) -> Inductor_SMD:L_0805_2012Metric
- L5: value L_Small -> 17n; footprint (none) -> Inductor_SMD:L_0603_1608Metric
- R35: value 330 -> 100
Connections:
- net GND: now also C8.2
- net at C32.2, C7.2, C9.1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: now also L13.2; no longer C8.2
- net at C1.1, C2.1, C3.1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: now also L10.1
- net at C3.2, C5.1, C6.1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: now also L10.2, L13.1
Other:
- moved on the sheet: C1, C5, C9, L1, L3, L5

Commit message: added test point for if filter
Parts:
- added J4, J5: UFL, Connector_Coaxial:U.FL_Molex_MCRF_73412-0110_Vertical, symbol Connector:Conn_Coaxial_Small
- added R49, R50, R51, R52: 0, Resistor_SMD:R_0402_1005Metric, symbol Device:R_Small
Connections:
- net GND: now also J4.2 (Ext), J5.2 (Ext)
- net at C7.2, C9.1, L13.2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: now also R49.1, R50.1; no longer C32.2
- net at C1.1, C2.1, C3.1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: now also R51.1, R52.1; no longer U7.2
- new net: J4.1 (In), R50.2
- new net: J5.1 (In), R52.2
- new net: R51.2, U7.2
- new net: C32.2, R49.2
Other:
- moved on the sheet: C1, C2, C3, C5, C6, C7, C8, C9, L1, L10, L13, L2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
