File: de1-sdr.kicad_pcb (KiCad board)
At the start: 2 copper layers, 0 parts

Commit message: fixed IF filter. todo: fix matching networks
Parts:
- added C1: 120p, Capacitor_SMD:C_0402_1005Metric, F.Cu at (168.1, 115.1)
- added C10: 100p, Capacitor_SMD:C_0402_1005Metric, F.Cu at (168.1, 122.9)
- added C11: 100p, Capacitor_SMD:C_0402_1005Metric, F.Cu at (168.1, 124.9)
- added C12: 100p, Capacitor_SMD:C_0402_1005Metric, F.Cu at (168.1, 126.9)
- added C13: 100p, Capacitor_SMD:C_0402_1005Metric, F.Cu at (168.1, 128.8)
- added C14: 1u, Capacitor_SMD:C_0402_1005Metric, F.Cu at (171.0, 115.1)
- added C15: 100p, Capacitor_SMD:C_0402_1005Metric, F.Cu at (171.0, 117.0)
- added C16: 100p, Capacitor_SMD:C_0402_1005Metric, F.Cu at (171.0, 119.0)
- added C17: 1u, Capacitor_SMD:C_0402_1005Metric, F.Cu at (171.0, 121.0)
- added C18: 100p, Capacitor_SMD:C_0402_1005Metric, F.Cu at (171.0, 122.9)
- added C19: 1u, Capacitor_SMD:C_0402_1005Metric, F.Cu at (171.0, 124.9)
- added C2: 6.4p, Capacitor_SMD:C_0402_1005Metric, F.Cu at (168.1, 117.0)
- added C20: 100p, Capacitor_SMD:C_0402_1005Metric, F.Cu at (171.0, 126.9)
- added C21: 1u, Capacitor_SMD:C_0402_1005Metric, F.Cu at (171.0, 128.8)
- added C22: 100p, Capacitor_SMD:C_0402_1005Metric, F.Cu at (173.9, 115.1)
- added C23: 270p, Capacitor_SMD:C_0402_1005Metric, F.Cu at (173.9, 117.0)
- added C24: 15p, Capacitor_SMD:C_0402_1005Metric, F.Cu at (173.9, 119.0)
- added C25: 100p, Capacitor_SMD:C_0402_1005Metric, F.Cu at (173.9, 121.0)
- added C26: 100p, Capacitor_SMD:C_0402_1005Metric, F.Cu at (173.9, 122.9)
- added C27: 100p, Capacitor_SMD:C_0402_1005Metric, F.Cu at (173.9, 124.9)
- added C28: 100p, Capacitor_SMD:C_0402_1005Metric, F.Cu at (173.9, 126.9)
- added C29: 100p, Capacitor_SMD:C_0402_1005Metric, F.Cu at (173.9, 128.8)
- added C3: 220p, Capacitor_SMD:C_0402_1005Metric, F.Cu at (168.1, 119.0)
- added C30: 10n, Capacitor_SMD:C_0402_1005Metric, F.Cu at (176.7, 115.1)
- added C31: 10u, Capacitor_SMD:C_0603_1608Metric, F.Cu at (168.7, 75.9)
- added C32: 10n, Capacitor_SMD:C_0402_1005Metric, F.Cu at (176.7, 117.0)
- added C33: 10u, Capacitor_SMD:C_0603_1608Metric, F.Cu at (168.7, 78.4)
- added C34: DNI, Capacitor_SMD:C_0402_1005Metric, F.Cu at (176.7, 119.0)
- added C35: 10n, Capacitor_SMD:C_0402_1005Metric, F.Cu at (176.7, 121.0)
- added C36: 100p, Capacitor_SMD:C_0402_1005Metric, F.Cu at (176.7, 122.9)
- added C37: 10u, Capacitor_SMD:C_0603_1608Metric, F.Cu at (168.7, 80.9)
- added C38: 10u, Capacitor_SMD:C_0603_1608Metric, F.Cu at (168.7, 83.4)
- added C39: 100p, Capacitor_SMD:C_0402_1005Metric, F.Cu at (176.7, 124.9)
- added C4: 6.4p, Capacitor_SMD:C_0402_1005Metric, F.Cu at (168.1, 121.0)
- added C40: 10u, Capacitor_SMD:C_0603_1608Metric, F.Cu at (168.7, 85.9)
- added C41: 100n, Capacitor_SMD:C_0402_1005Metric, F.Cu at (176.7, 126.9)
- added C42: 100n, Capacitor_SMD:C_0402_1005Metric, F.Cu at (176.7, 128.8)
- added C43: 100n, Capacitor_SMD:C_0402_1005Metric, F.Cu at (179.6, 115.1)
- added C44: 100n, Capacitor_SMD:C_0402_1005Metric, F.Cu at (179.6, 117.0)
- added C45: 10u, Capacitor_SMD:C_0603_1608Metric, F.Cu at (168.7, 88.4)
- added C46: 100n, Capacitor_SMD:C_0402_1005Metric, F.Cu at (179.6, 119.0)
- added C47: 100n, Capacitor_SMD:C_0402_1005Metric, F.Cu at (179.6, 121.0)
- added C48: 1u, Capacitor_SMD:C_0603_1608Metric, F.Cu at (168.7, 90.9)
- added C49: 100n, Capacitor_SMD:C_0402_1005Metric, F.Cu at (179.6, 122.9)
- added C5: 160p, Capacitor_SMD:C_0603_1608Metric, F.Cu at (168.7, 73.4)
- added C50: 100n, Capacitor_SMD:C_0402_1005Metric, F.Cu at (179.6, 124.9)
- added C51: 100n, Capacitor_SMD:C_0402_1005Metric, F.Cu at (179.6, 126.9)
- added C52: 1u, Capacitor_SMD:C_0603_1608Metric, F.Cu at (172.7, 73.4)
- added C53: 10u, Capacitor_SMD:C_0603_1608Metric, F.Cu at (172.7, 75.9)
- added C54: 100n, Capacitor_SMD:C_0402_1005Metric, F.Cu at (179.6, 128.8)
- added C55: 10u, Capacitor_SMD:C_0603_1608Metric, F.Cu at (172.7, 78.4)
- added C56: 10n, Capacitor_SMD:C_0402_1005Metric, F.Cu at (182.5, 115.1)
- added C57: 0.47u, Capacitor_SMD:C_0603_1608Metric, F.Cu at (172.7, 80.9)
- added C58: 10u, Capacitor_SMD:C_0603_1608Metric, F.Cu at (172.7, 83.4)
- added C59: 1u, Capacitor_SMD:C_0603_1608Metric, F.Cu at (172.7, 85.9)
- added C60: 1u, Capacitor_SMD:C_0603_1608Metric, F.Cu at (172.7, 88.4)
- added C61: 1u, Capacitor_SMD:C_0603_1608Metric, F.Cu at (172.7, 90.9)
- added C62: 1u, Capacitor_SMD:C_0603_1608Metric, F.Cu at (176.7, 73.4)
- added C63: 1u, Capacitor_SMD:C_0603_1608Metric, F.Cu at (176.7, 75.9)
- added C64: 1u, Capacitor_SMD:C_0603_1608Metric, F.Cu at (176.7, 78.4)
- added C65: 100n, Capacitor_SMD:C_0402_1005Metric, F.Cu at (182.5, 117.0)
- added C66: ~, Capacitor_SMD:C_0402_1005Metric, F.Cu at (182.5, 119.0)
- added C67: 220n, Capacitor_SMD:C_0402_1005Metric, F.Cu at (182.5, 121.0)
- added C68: ~, Capacitor_SMD:C_0402_1005Metric, F.Cu at (182.5, 122.9)
- added C69: 1.5n, Capacitor_SMD:C_0402_1005Metric, F.Cu at (182.5, 124.9)
- added C70: 100n, Capacitor_SMD:C_0402_1005Metric, F.Cu at (182.5, 126.9)
- added C71: 100n, Capacitor_SMD:C_0402_1005Metric, F.Cu at (182.5, 128.8)
- added C72: 10u, Capacitor_SMD:C_0603_1608Metric, F.Cu at (176.7, 80.9)
- added C73: 1u, Capacitor_SMD:C_0603_1608Metric, F.Cu at (176.7, 83.4)
- added C74: 10u, Capacitor_SMD:C_0603_1608Metric, F.Cu at (176.7, 85.9)
- added C75: 1u, Capacitor_SMD:C_0603_1608Metric, F.Cu at (176.7, 88.4)
- added C76: 10u, Capacitor_SMD:C_0603_1608Metric, F.Cu at (176.7, 90.9)
- added C77: 1u, Capacitor_SMD:C_0603_1608Metric, F.Cu at (180.7, 73.4)
- added C78: 10u, Capacitor_SMD:C_0603_1608Metric, F.Cu at (180.7, 75.9)
- added C79: 1u, Capacitor_SMD:C_0603_1608Metric, F.Cu at (180.7, 78.4)
- added C80: 10u, Capacitor_SMD:C_0603_1608Metric, F.Cu at (180.7, 80.9)
- added C81: 1u, Capacitor_SMD:C_0603_1608Metric, F.Cu at (180.7, 83.4)
- added C82: 10u, Capacitor_SMD:C_0603_1608Metric, F.Cu at (180.7, 85.9)
- added C83: 10u, Capacitor_SMD:C_0603_1608Metric, F.Cu at (180.7, 88.4)
- added C84: 10u, Capacitor_SMD:C_0603_1608Metric, F.Cu at (180.7, 90.9)
- added C85: 10u, Capacitor_SMD:C_0603_1608Metric, F.Cu at (184.7, 73.4)
- added FB1: BLF03JD421GZED, Inductor_SMD:L_0201_0603Metric, F.Cu at (201.6, 93.1)
- added FB10: BLM15PX221SN1D, Inductor_SMD:L_0402_1005Metric, F.Cu at (168.1, 95.2)
- added FB11: BLM15PX221SN1D, Inductor_SMD:L_0402_1005Metric, F.Cu at (168.1, 97.2)
- added FB12: BLM15PX221SN1D, Inductor_SMD:L_0402_1005Metric, F.Cu at (168.1, 99.1)
- added FB13: BLM15PX221SN1D, Inductor_SMD:L_0402_1005Metric, F.Cu at (168.1, 101.1)
- added FB14: BLM15PX221SN1D, Inductor_SMD:L_0402_1005Metric, F.Cu at (168.1, 103.1)
- added FB15: BLM15PX221SN1D, Inductor_SMD:L_0402_1005Metric, F.Cu at (168.1, 105.1)
- added FB2: BLF03JD421GZED, Inductor_SMD:L_0201_0603Metric, F.Cu at (201.6, 94.8)
- added FB3: BLF03JD421GZED, Inductor_SMD:L_0201_0603Metric, F.Cu at (201.6, 96.6)
- added FB4: BLF03JD421GZED, Inductor_SMD:L_0201_0603Metric, F.Cu at (201.6, 98.3)
- added FB5: BLF03JD421GZED, Inductor_SMD:L_0201_0603Metric, F.Cu at (201.6, 100.1)
- added FB6: BLF03JD421GZED, Inductor_SMD:L_0201_0603Metric, F.Cu at (201.6, 101.8)
- added FB7: BLF03JD421GZED, Inductor_SMD:L_0201_0603Metric, F.Cu at (201.6, 103.6)
- added FB8: BLF03JD421GZED, Inductor_SMD:L_0201_0603Metric, F.Cu at (201.6, 105.3)
- added FB9: BLM15PX221SN1D, Inductor_SMD:L_0402_1005Metric, F.Cu at (168.1, 93.2)
- added FL1: B39162B8813P810, Filter:Filter_1109-5_1.1x0.9mm, F.Cu at (203.3, 73.2)
- added FL2: DEA162025LT-5046E1, 0thaumati-footprintslib:FILTER_TDK_0402, F.Cu at (203.3, 78.1)
- added FL3: B39162B8813P810, Filter:Filter_1109-5_1.1x0.9mm, F.Cu at (203.3, 75.7)
- added J1: RF IN, 0thaumati-footprintslib:ADAMTECH_RF2-143-T-17-50-G, F.Cu at (193.8, 97.7)
- added J2: DE1-HEADER, Connector_IDC:IDC-Header_2x20_P2.54mm_Vertical, F.Cu at (159.9, 78.2)
- added J3: UFL, Connector_Coaxial:U.FL_Molex_MCRF_73412-0110_Vertical, F.Cu at (192.3, 111.1)
- added J4: UFL, Connector_Coaxial:U.FL_Molex_MCRF_73412-0110_Vertical, F.Cu at (192.3, 117.1)
- added J5: UFL, Connector_Coaxial:U.FL_Molex_MCRF_73412-0110_Vertical, F.Cu at (192.3, 123.2)
- added L1: 20n, Inductor_SMD:L_0603_1608Metric, F.Cu at (184.7, 75.9)
- added L11: 1u, Inductor_SMD:L_1008_2520Metric, F.Cu at (186.6, 121.8)
- added L12: 1u, Inductor_SMD:L_1008_2520Metric, F.Cu at (186.6, 125.6)
- added L2: 390n, Inductor_SMD:L_0603_1608Metric, F.Cu at (184.7, 78.4)
- added L3: 11n, Inductor_SMD:L_0603_1608Metric, F.Cu at (184.7, 80.9)
- added L4: 390n, Inductor_SMD:L_0603_1608Metric, F.Cu at (184.7, 83.4)
- added L5: 16n, Capacitor_SMD:C_0603_1608Metric, F.Cu at (184.7, 85.9)
- added L6: AC5037SQ-68NJ, Inductor_SMD:L_1812_4532Metric_Pad1.30x3.40mm_HandSolder, F.Cu at (198.1, 74.6)
- added L7: 18n, Inductor_SMD:L_0805_2012Metric, F.Cu at (193.9, 90.7)
- added L8: 2.2n, Inductor_SMD:L_0402_1005Metric, F.Cu at (168.1, 107.1)
- added L9: 330n, Inductor_SMD:L_0402_1005Metric, F.Cu at (168.1, 109.1)
- added Q1: BSS138, Package_TO_SOT_SMD:SOT-23, F.Cu at (189.2, 81.6)
- added Q2: AO3401A, Package_TO_SOT_SMD:SOT-23, F.Cu at (189.2, 86.1)
- added R10: 1k, Resistor_SMD:R_0402_1005Metric, F.Cu at (171.0, 105.1)
- added R11: 1k, Resistor_SMD:R_0402_1005Metric, F.Cu at (171.0, 107.1)
- added R12: 1k, Resistor_SMD:R_0402_1005Metric, F.Cu at (171.0, 109.1)
- added R13: 1k, Resistor_SMD:R_0402_1005Metric, F.Cu at (171.0, 111.1)
- added R14: 1k, Resistor_SMD:R_0402_1005Metric, F.Cu at (171.0, 113.1)
- added R15: 1k, Resistor_SMD:R_0402_1005Metric, F.Cu at (174.0, 93.2)
- added R16: 100, Resistor_SMD:R_0402_1005Metric, F.Cu at (174.0, 95.2)
- added R17: 100, Resistor_SMD:R_0402_1005Metric, F.Cu at (174.0, 97.2)
- added R18: 0, Resistor_SMD:R_0402_1005Metric, F.Cu at (174.0, 99.1)
- added R19: 10k, Resistor_SMD:R_0402_1005Metric, F.Cu at (174.0, 101.1)
- added R2: 100k, Resistor_SMD:R_0402_1005Metric, F.Cu at (168.1, 111.1)
- added R20: 22, Resistor_SMD:R_0402_1005Metric, F.Cu at (174.0, 103.1)
- added R21: 22, Resistor_SMD:R_0402_1005Metric, F.Cu at (174.0, 105.1)
- added R22: 22, Resistor_SMD:R_0402_1005Metric, F.Cu at (174.0, 107.1)
- added R23: 22, Resistor_SMD:R_0402_1005Metric, F.Cu at (174.0, 109.1)
- added R24: 22, Resistor_SMD:R_0402_1005Metric, F.Cu at (174.0, 111.1)
- added R25: 22, Resistor_SMD:R_0402_1005Metric, F.Cu at (174.0, 113.1)
- added R26: 22, Resistor_SMD:R_0402_1005Metric, F.Cu at (176.9, 93.2)
- added R27: 22, Resistor_SMD:R_0402_1005Metric, F.Cu at (176.9, 95.2)
- added R28: 22, Resistor_SMD:R_0402_1005Metric, F.Cu at (176.9, 97.2)
- added R29: 22, Resistor_SMD:R_0402_1005Metric, F.Cu at (176.9, 99.1)
- added R3: 3.3k, Resistor_SMD:R_0402_1005Metric, F.Cu at (168.1, 113.1)
- added R30: 22, Resistor_SMD:R_0402_1005Metric, F.Cu at (176.9, 101.1)
- added R31: 22, Resistor_SMD:R_0402_1005Metric, F.Cu at (176.9, 103.1)
- added R32: 22, Resistor_SMD:R_0402_1005Metric, F.Cu at (176.9, 105.1)
- added R33: 200, Resistor_SMD:R_0402_1005Metric, F.Cu at (176.9, 107.1)
- added R34: 22, Resistor_SMD:R_0402_1005Metric, F.Cu at (176.9, 109.1)
- added R35: 100, Resistor_SMD:R_0402_1005Metric, F.Cu at (176.9, 111.1)
- added R36: 0, Resistor_SMD:R_0402_1005Metric, F.Cu at (176.9, 113.1)
- added R37: 0, Resistor_SMD:R_0402_1005Metric, F.Cu at (179.8, 93.2)
- added R38: 51, Resistor_SMD:R_0402_1005Metric, F.Cu at (179.8, 95.2)
- added R39: 51, Resistor_SMD:R_0402_1005Metric, F.Cu at (179.8, 97.2)
- added R4: 1k, Resistor_SMD:R_0402_1005Metric, F.Cu at (171.0, 93.2)
- added R40: 1k, Resistor_SMD:R_0402_1005Metric, F.Cu at (179.8, 99.1)
- added R41: 1k, Resistor_SMD:R_0402_1005Metric, F.Cu at (179.8, 101.1)
- added R42: 1k, Resistor_SMD:R_0402_1005Metric, F.Cu at (179.8, 103.1)
- added R43: 1k, Resistor_SMD:R_0402_1005Metric, F.Cu at (179.8, 105.1)
- added R44: 1k, Resistor_SMD:R_0402_1005Metric, F.Cu at (179.8, 107.1)
- added R45: 1k, Resistor_SMD:R_0402_1005Metric, F.Cu at (179.8, 109.1)
- added R46: 1k, Resistor_SMD:R_0402_1005Metric, F.Cu at (179.8, 111.1)
- added R47: 100k, Resistor_SMD:R_0402_1005Metric, F.Cu at (179.8, 113.1)
- added R48: 100k, Resistor_SMD:R_0402_1005Metric, F.Cu at (182.7, 93.2)
- added R49: 0, Resistor_SMD:R_0402_1005Metric, F.Cu at (182.7, 95.2)
- added R5: 1k, Resistor_SMD:R_0402_1005Metric, F.Cu at (171.0, 95.2)
- added R50: 0, Resistor_SMD:R_0402_1005Metric, F.Cu at (182.7, 97.2)
- added R51: 0, Resistor_SMD:R_0402_1005Metric, F.Cu at (182.7, 99.1)
- added R52: 0, Resistor_SMD:R_0402_1005Metric, F.Cu at (182.7, 101.1)
- added R6: 1k, Resistor_SMD:R_0402_1005Metric, F.Cu at (171.0, 97.2)
- added R7: 1k, Resistor_SMD:R_0402_1005Metric, F.Cu at (171.0, 99.1)
- added R8: 1k, Resistor_SMD:R_0402_1005Metric, F.Cu at (171.0, 101.1)
- added R9: 1k, Resistor_SMD:R_0402_1005Metric, F.Cu at (171.0, 103.1)
- added T1: TC4-1TX+, Transformer_SMD:Transformer_MiniCircuits_AT224-1A, F.Cu at (201.1, 88.0)
- added U1: AD9609-80, Package_DFN_QFN:QFN-32-1EP_5x5mm_P0.5mm_EP3.45x3.45mm, F.Cu at (190.8, 75.8)
- added U10: TPS7A2018DBV, Package_TO_SOT_SMD:SOT-23-5, F.Cu at (186.7, 103.8)
- added U11: TPS7A2033DBV, Package_TO_SOT_SMD:SOT-23-5, F.Cu at (186.7, 108.5)
- added U12: TPS7A2033DBV, Package_TO_SOT_SMD:SOT-23-5, F.Cu at (186.7, 113.1)
- added U13: TPS7A2033DBV, Package_TO_SOT_SMD:SOT-23-5, F.Cu at (186.7, 117.7)
- added U2: QPL9547, Package_DFN_QFN:DFN-8-1EP_2x2mm_P0.5mm_EP0.8x1.6mm, F.Cu at (186.3, 129.3)
- added U3: MAX2682, Package_TO_SOT_SMD:SOT-23-6, F.Cu at (186.7, 94.6)
- added U4: LMX2572, Package_DFN_QFN:HVQFN-40-1EP_6x6mm_P0.5mm_EP4.1x4.1mm, F.Cu at (199.9, 124.4)
- added U5: BDA4620, Package_DFN_QFN:QFN-20-1EP_4x4mm_P0.5mm_EP2.5x2.5mm, F.Cu at (195.1, 82.5)
- added U6: TPS7A2018DBV, Package_TO_SOT_SMD:SOT-23-5, F.Cu at (186.7, 99.2)
- added U7: PAT1220-C-2DB, RF_Converter:RF_Attenuator_Susumu_PAT1220, F.Cu at (193.9, 87.6)
- added U8: BG18C, Package_TO_SOT_SMD:SOT-89-3, F.Cu at (198.7, 111.0)
- added U9: BG18C, Package_TO_SOT_SMD:SOT-89-3, F.Cu at (198.7, 117.2)
- added Y1: ECS-3518-800-B-TR, Oscillator:Oscillator_SMD_EuroQuartz_XO53-4Pin_5.0x3.2mm, F.Cu at (201.8, 82.0)

Commit message: start placement
Parts:
- removed C18: 100p, Capacitor_SMD:C_0402_1005Metric
- removed R14: 1k, Resistor_SMD:R_0402_1005Metric
- added C6: 27p, Capacitor_SMD:C_0402_1005Metric, F.Cu at (125.5, 104.5)
- added C7: 130p, Capacitor_SMD:C_0402_1005Metric, F.Cu at (131.5, 100.0)
- added C8: 10u, Capacitor_SMD:C_0603_1608Metric, F.Cu at (147.5, 116.5)
- added C86: 100p, Capacitor_SMD:C_0402_1005Metric, F.Cu at (153.5, 105.5)
- added C9: 1u, Capacitor_SMD:C_0402_1005Metric, F.Cu at (151.5, 81.5)
- added D1: ESD601DPYRQ1, Diode_SMD:D_0402_1005Metric, F.Cu at (153.0, 89.0)
- added D2: LED, LED_SMD:LED_0603_1608Metric, F.Cu at (117.5, 97.0)
- added D3: LED, LED_SMD:LED_0603_1608Metric, F.Cu at (117.5, 102.0)
- added D4: LED, LED_SMD:LED_0603_1608Metric, F.Cu at (117.5, 99.5)
- added L10: 330n, Inductor_SMD:L_1008_2520Metric, F.Cu at (128.0, 105.5)
- added L13: 62n, Inductor_SMD:L_0603_1608Metric, F.Cu at (131.5, 101.5)
- added R1: 1k, Resistor_SMD:R_0201_0603Metric, F.Cu at (144.0, 108.5)
- added R53: 0, Resistor_SMD:R_0402_1005Metric, F.Cu at (149.5, 112.0)
- added R54: 0, Resistor_SMD:R_0402_1005Metric, F.Cu at (156.0, 107.5)
- added R55: ~, Resistor_SMD:R_0402_1005Metric, F.Cu at (156.5, 112.0)
- added R56: 1k, Resistor_SMD:R_0402_1005Metric, F.Cu at (120.5, 97.0)
- added R57: 1k, Resistor_SMD:R_0402_1005Metric, F.Cu at (120.5, 102.0)
- added R58: 1k, Resistor_SMD:R_0402_1005Metric, F.Cu at (120.5, 99.5)
- C1: value 120p -> 91p
- C2: value 6.4p -> 62p
- C23: value 270p -> ~
- C24: value 15p -> ~
- C3: value 220p -> 36p
- C34: value DNI -> 10p
- C4: value 6.4p -> 180p
- C5: value 160p -> 22p; footprint Capacitor_SMD:C_0603_1608Metric -> Capacitor_SMD:C_0402_1005Metric
- L1: value 20n -> 82n; footprint Inductor_SMD:L_0603_1608Metric -> Inductor_SMD:L_0805_2012Metric
- L11, L12: value 1u -> 2.7u; footprint Inductor_SMD:L_1008_2520Metric -> Inductor_SMD:L_1210_3225Metric
- L2: value 390n -> 220n; footprint Inductor_SMD:L_0603_1608Metric -> Inductor_SMD:L_0805_2012Metric
- L3: value 11n -> 130n; footprint Inductor_SMD:L_0603_1608Metric -> Inductor_SMD:L_0805_2012Metric
- L4: value 390n -> 43n
- L5: value 16n -> 300n; footprint Capacitor_SMD:C_0603_1608Metric -> Inductor_SMD:L_0805_2012Metric
- L6: footprint Inductor_SMD:L_1812_4532Metric_Pad1.30x3.40mm_HandSolder -> 0thaumati-footprintslib:AC5037SQ-68NJ
- L8: value 2.2n -> ~
- L9: value 330n -> ~; footprint Inductor_SMD:L_0402_1005Metric -> Inductor_SMD:L_0805_2012Metric
- R10, R11, R12, R13, R20, R21, R22, R23, R24, R25, R26, R27, R28, R29, R30, R31, R32, R5, R6, R7, R8, R9: footprint Resistor_SMD:R_0402_1005Metric -> Resistor_SMD:R_0201_0603Metric
- R16, R17: value 100 -> 33
- R46: value 1k -> 1.2k
- moved FB7 103.4 mm to (98.5, 112.1), turned to 180 degrees
- moved FB6 100.6 mm to (102.5, 119.1), turned to 180 degrees
- moved FB3 99.5 mm to (102.5, 105.6), turned to 90 degrees
- moved FB5 97.9 mm to (106.0, 121.1), turned to -90 degrees
- moved U4 94.1 mm to (106.5, 113.0)
- moved FL2 93.9 mm to (116.5, 114.1), turned to 180 degrees
- moved C51 90.8 mm to (104.0, 76.5), turned to 90 degrees
- moved C44 90.4 mm to (96.5, 81.5)
- moved C41 89.3 mm to (103.0, 76.5), turned to -90 degrees
- moved C50 88.9 mm to (105.0, 76.5), turned to 90 degrees
- moved FB8 88.9 mm to (114.0, 120.6)
- moved FB4 88.5 mm to (114.0, 111.1)
- moved U1 88.5 mm to (102.5, 82.0), turned to -90 degrees
- moved C52 86.8 mm to (98.0, 117.6)
- moved J2 86.4 mm to (86.8, 124.1), turned to 180 degrees
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Connections:
- C2 pad 1: Net-(C2-Pad1) -> Net-(C1-Pad1)
- C21 pad 2: +3V3_A -> Net-(Q2-D)
- C23 pad 1: Net-(U5-RF2) -> GND
- C23 pad 2: Net-(U3-RFIN) -> Net-(C23-Pad2)
- C24 pad 1: Net-(U3-IFOUT) -> Net-(C24-Pad1)
- C3 pad 1: Net-(C2-Pad2) -> Net-(C3-Pad1)
- C3 pad 2: GND -> Net-(C2-Pad2)
- C34 pad 1: /ADC_INP -> /ADC_INM
- C34 pad 2: /ADC_INM -> /ADC_INP
- C4 pad 1: Net-(C4-Pad1) -> Net-(C2-Pad2)
- C4 pad 2: Net-(C4-Pad2) -> GND
- C5 pad 1: Net-(C4-Pad2) -> Net-(C2-Pad2)
- C5 pad 2: GND -> Net-(C5-Pad2)
- J2 pad 4: unconnected-(J2-Pin_4-Pad4) -> /LED1
- L2 pad 2: Net-(C2-Pad1) -> Net-(C3-Pad1)
- L3 pad 1: Net-(C2-Pad2) -> Net-(C1-Pad1)
- L3 pad 2: GND -> Net-(C2-Pad2)
- L4 pad 2: Net-(C4-Pad1) -> GND
- L5 pad 1: Net-(C4-Pad2) -> Net-(C2-Pad2)
- L5 pad 2: GND -> Net-(C6-Pad1)
- L8 pad 1: Net-(U5-RF2) -> Net-(C23-Pad2)
- L8 pad 2: GND -> Net-(U3-RFIN)
- L9 pad 2: Net-(U3-IFOUT) -> Net-(C24-Pad1)
- R10 pad 1: Net-(U5-D5) -> Net-(U5-D2)
- R10 pad 2: /DSA_D5 -> /DSA_D2
- R11 pad 1: Net-(U5-P/S) -> Net-(U5-D3)
- R11 pad 2: GND -> /DSA_D3
- R12 pad 1: Net-(U5-SERIN) -> Net-(U5-D4)
- R12 pad 2: GND -> /DSA_D4
- R13 pad 1: Net-(U5-CLK) -> Net-(U5-D5)
- R13 pad 2: GND -> /DSA_D5
- R16 pad 1: /ADC_INP -> /ADC_INM
- R17 pad 1: /ADC_INM -> /ADC_INP
- R49 pad 1: Net-(C4-Pad2) -> Net-(C5-Pad2)
- R5 pad 1: Net-(U5-D0) -> Net-(U5-CLK)
- R5 pad 2: /DSA_D0 -> GND
- R50 pad 1: Net-(C4-Pad2) -> Net-(C5-Pad2)
- R6 pad 1: Net-(U5-D1) -> Net-(U5-SERIN)
- R6 pad 2: /DSA_D1 -> GND
- R7 pad 1: Net-(U5-D2) -> Net-(U5-P/S)
- R7 pad 2: /DSA_D2 -> GND
- R8 pad 1: Net-(U5-D3) -> Net-(U5-D0)
- R8 pad 2: /DSA_D3 -> /DSA_D0
- R9 pad 1: Net-(U5-D4) -> Net-(U5-D1)
- R9 pad 2: /DSA_D4 -> /DSA_D1
Other:
- board outline added: 80 x 60 mm

Commit message: routed pcb
Parts:
- moved C72 8.25 mm to (120.4, 73.7)
- moved C73 8.25 mm to (126.9, 73.7)
- moved C82 8.25 mm to (133.2, 74.2)
- moved C83 8.25 mm to (135.2, 74.2)
- moved C84 8.25 mm to (137.2, 74.2)
- moved C85 8.25 mm to (139.2, 74.2)
- moved FB14 8.25 mm to (132.2, 72.2)
- moved FB15 8.25 mm to (136.2, 72.2)
- moved FB9 8.25 mm to (118.2, 72.8)
- moved U6 8.25 mm to (123.8, 73.8)
- moved C43 6.17 mm to (113.8, 80.8)
- moved R19 6.17 mm to (113.8, 81.8)
- moved C41 5.37 mm to (107.8, 74.0)
- moved C34 5.26 mm to (111.8, 78.8)
- moved C40 5.26 mm to (112.8, 75.8)
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Connections:
- J2 pad 1: /ADC_DCO -> /LNA_EN
- J2 pad 11: +5V_IN -> unconnected-(J2-Pin_11-Pad11)
- J2 pad 13: /ADC_SPI_SDIO -> /DSA_D1
- J2 pad 15: /PLL_MUXOUT -> /DSA_D0
- J2 pad 17: /PLL_EN -> /PLL_SPI_CS
- J2 pad 19: /PLL_SPI_SCLK -> /PLL_SPI_MOSI
- J2 pad 2: /MIXER_SHDN -> /ANT_PWR_EN
- J2 pad 21: /PLL_SPI_MOSI -> /PLL_SPI_SCLK
- J2 pad 23: /PLL_SPI_CS -> /PLL_EN
- J2 pad 25: /DSA_D0 -> /PLL_MUXOUT
- J2 pad 27: /DSA_D1 -> /ADC_SPI_SDIO
- J2 pad 29: unconnected-(J2-Pin_29-Pad29) -> +5V_IN
- J2 pad 3: unconnected-(J2-Pin_3-Pad3) -> /DSA_D5
- J2 pad 31: /DSA_D2 -> /ADC_SPI_SCLK
- J2 pad 33: /DSA_D3 -> /ADC_SPI_CS
- J2 pad 35: /DSA_D4 -> /ADC_MODE_OR
- J2 pad 37: /DSA_D5 -> unconnected-(J2-Pin_37-Pad37)
- J2 pad 38: /XO_EN -> /LED1
- J2 pad 39: /LNA_EN -> /ADC_DCO
- J2 pad 4: /LED1 -> /XO_EN
- J2 pad 40: /ANT_PWR_EN -> /MIXER_SHDN
- J2 pad 5: /ADC_MODE_OR -> /DSA_D4
- J2 pad 7: /ADC_SPI_CS -> /DSA_D3
- J2 pad 9: /ADC_SPI_SCLK -> /DSA_D2
Routing:
- net +5V_IN: track 0.00 -> 135.7 mm, vias 0 -> 8
- net +3V3: track 0.00 -> 113.6 mm, vias 0 -> 11
- net /MIXER_SHDN: track 0.00 -> 101.1 mm, vias 0 -> 3
- net /ANT_PWR_EN: track 0.00 -> 96.1 mm, vias 0 -> 2
- net +5V_A: track 0.00 -> 80.4 mm, vias 0 -> 3
- net /DSA_D0: track 0.00 -> 79.9 mm, vias 0 -> 1
- net /DSA_D1: track 0.00 -> 79.4 mm, vias 0 -> 1
- net /DSA_D4: track 0.00 -> 78.1 mm, vias 0 -> 1
- net /DSA_D3: track 0.00 -> 77.9 mm, vias 0 -> 1
- net /DSA_D2: track 0.00 -> 77.3 mm, vias 0 -> 1
- net /LNA_EN: track 0.00 -> 73.0 mm, vias 0 -> 2
- net /DSA_D5: track 0.00 -> 68.2 mm, vias 0 -> 1
- net /PLL_SPI_SCLK: track 0.00 -> 57.1 mm, vias 0 -> 1
- net /LED1: track 0.00 -> 56.5 mm, vias 0 -> 5
- net /LO_L1: track 0.00 -> 54.3 mm
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- added copper zone on In2.Cu, net +1V8_ADC
- added copper zone on In2.Cu, net +3V3
- added copper zone on B.Cu, net GND
- added copper zone on F.Cu, net GND
- added copper zone on In1.Cu, net GND
- added copper zone on In2.Cu, net GND
Other:
- copper layers 2 -> 4

Commit message: finished routing
Routing:
- net GND: vias 524 -> 531
Other:
- outline, holes or cut-outs redrawn
Changed lines of the file:
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@@
 		(capping no)
 		(filling no)
-		(zone_defaults)
 		(pcbplotparams
 			(layerselection 0x00000000_00000000_55555555_5755f5ff)
@@
 		(layer "Edge.Cuts")
 	)
+	(gr_circle
+		(center 156 73)
+		(end 158 73)
+		(stroke
+			(width 0.05)
+			(type default)
+		)
+		(fill no)
+		(layer "Edge.Cuts")
+	)
+	(gr_circle
+		(center 156 127)
+		(end 158 127)
+		(stroke
+			(width 0.05)
+			(type default)
+		)
+		(fill no)
+		(layer "Edge.Cuts")
+	)
 	(segment
 		(start 113.48 116.56676)
@@
 	)
 	(via
-		(at 79.75 72.75)
+		(at 80.25 73)
 		(size 0.6)
 		(drill 0.3)
@@
 	)
 	(via
-		(at 157.25 126.25)
+		(at 156.75 79)
 		(size 0.6)
 		(drill 0.3)
@@
 	)
 	(via
+		(at 88.25 73.25)
+		(size 0.6)
+		(drill 0.3)
+		(layers "F.Cu" "B.Cu")
+		(free yes)
+		(net "GND")
+	)
+	(via
 		(at 114 87.75)
 		(size 0.6)
@@
 	)
 	(via
-		(at 154 108.5)
+		(at 153.75 108.75)
 		(size 0.6)
 		(drill 0.3)
@@
 	)
 	(via
-		(at 155.25 127.5)
+		(at 139.75 76.5)
 		(size 0.6)
 		(drill 0.3)
@@
 	)
 	(via
-		(at 139.75 76.5)
+		(at 92 111.25)
 		(size 0.6)
 		(drill 0.3)
@@
 	)
 	(via
-		(at 92 111.25)
+		(at 157.25 97)
 		(size 0.6)
 		(drill 0.3)
@@
 	)
 	(via
-		(at 157.25 97)
+		(at 157.5 79.75)
 		(size 0.6)
 		(drill 0.3)
@@
 	)
 	(via
+		(at 154 125.25)
+		(size 0.6)
+		(drill 0.3)
+		(layers "F.Cu" "B.Cu")
+		(free yes)
+		(net "GND")
+	)
+	(via
 		(at 104 112.75)
 		(size 0.6)
@@
 	)
 	(via
+		(at 157.5 120.25)
+		(size 0.6)
+		(drill 0.3)
+		(layers "F.Cu" "B.Cu")
+		(free yes)
+		(net "GND")
+	)
+	(via
 		(at 102 98.5)
 		(size 0.6)
@@
 	)
 	(via
+		(at 147.25 72)
+		(size 0.6)
+		(drill 0.3)
+		(layers "F.Cu" "B.Cu")
+		(free yes)
+		(net "GND")
+	)
+	(via
 		(at 99.5 77.25)
 		(size 0.6)
@@
 	)
 	(via
+		(at 149 128.5)
+		(size 0.6)
+		(drill 0.3)
+		(layers "F.Cu" "B.Cu")
+		(free yes)
+		(net "GND")
+	)
+	(via
 		(at 128.25 87)
 		(size 0.6)
@@
 	)
 	(via
+		(at 157.25 117.25)
+		(size 0.6)
+		(drill 0.3)
+		(layers "F.Cu" "B.Cu")
+		(free yes)
+		(net "GND")
+	)
+	(via
 		(at 115 82.25)
 		(size 0.6)
@@
 	)
 	(via
+		(at 155.25 122.75)
+		(size 0.6)
+		(drill 0.3)
+		(layers "F.Cu" "B.Cu")
+		(free yes)
+		(net "GND")
+	)
+	(via
 		(at 151 128.25)
 		(size 0.6)
@@
 	)
 	(via
-		(at 153.75 126.75)
+		(at 152.5 127)
 		(size 0.6)
 		(drill 0.3)
@@
 	)
 	(via
-		(at 155.5 125)
+		(at 155.5 124)
 		(size 0.6)
 		(drill 0.3)
@@
 	)
 	(via
-		(at 79.75 120)
+		(at 80.5 120.75)
 		(size 0.6)
 		(drill 0.3)
